File: ProtoBoardSESmall/ProtoBoardSESmall.kicad_sch (KiCad schematic)
At the start: 35 parts, among them J1 TYPE-C-31-M-12, J10 BM05B-SRSS-TB_LF__SN_, J11 Conn_01x05_Female, J2 TYPE-C-31-M-12, J3 BM10B-SRSS-TB_LF__SN_, J4 Conn_01x05_Female, J5 BM05B-SRSS-TB_LF__SN_, J6 BM05B-SRSS-TB_LF__SN_, J7 Conn_01x05_Female, J8 BM05B-SRSS-TB_LF__SN_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

Commit message: Add lcsc references, routing wip
Parts:
- J10, J5, J6, J8, J9: Availability In Stock -> (none); Check_prices https://www.snapeda.com/parts/BM05B-SRSS-TB(LF)(SN)/JST+Sal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 -> (none); LCSC (none) -> C160391; MANUFACTURER JST Sales America Inc. -> (none); MAXIMUM_PACKAGE_HEIGHT 6.3 mm -> (none); MF JST Sales -> (none); MP BM05B-SRSS-TB(LF)(SN) -> (none); PARTREV N/A -> (none); Package None -> (none); Price None -> (none); SNAPEDA_PN BM05B-SRSS-TB(LF)(SN) -> (none); STANDARD Manufacturer Recommendations -> (none); SnapEDA_Link https://www.snapeda.com/parts/BM05B-SRSS-TB(LF)(SN)/JST+Sal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 -> (none)
- J3: Availability In Stock -> (none); Check_prices https://www.snapeda.com/parts/BM10B-SRSS-TB%20(LF)(SN)/JST/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 -> (none); LCSC (none) -> C160396; MAXIMUM_PACKAGE_HEIGHT 6.3 mm -> (none); MP BM10B-SRSS-TB (LF)(SN) -> (none); PARTREV N/A -> (none); Package None -> (none); Price None -> (none); SNAPEDA_PN BM10B-SRSS-TB(LF)(SN) -> (none); STANDARD Manufacturer Recommendations -> (none); SnapEDA_Link https://www.snapeda.com/parts/BM10B-SRSS-TB%20(LF)(SN)/JST/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 -> (none)
- U3: LCSC (none) -> C965555
Connections:
- net Servo1: now also J11.5 (Pin_5); no longer J11.1 (Pin_1)
- net Servo2: now also J11.4 (Pin_4); no longer J11.2 (Pin_2)
- net Servo4: now also J11.2 (Pin_2); no longer J11.4 (Pin_4)
- net Servo5: now also J11.1 (Pin_1); no longer J11.5 (Pin_5)

Commit message: Routing done + production files
Parts:
- added C7: 0.1uF, Capacitor_SMD:C_0402_1005Metric, symbol Device:C
- added TP1, TP5, TP6, TP7, TP8, TP9: TestPoint, TestPoint:TestPoint_Pad_D1.5mm, symbol Connector:TestPoint
Connections:
- net +3V3: now also U3.4 (VDD), C7.1, TP8.1
- net CH10: now also J5.4; no longer J5.3
- net CH11: now also J5.5; no longer J8.5
- net CH12: now also J8.5; no longer J8.4
- net CH13: now also J8.4; no longer J8.3
- net CH14: now also J8.3; no longer J9.3
- net CH15: now also J3.8; no longer J9.4
- net CH16: now also J9.3; no longer J9.5
- net CH7: now also J9.5; no longer J3.8
- net CH8: now also J9.4; no longer J5.5
- net CH9: now also J5.3; no longer J5.4
- net GND: now also U3.2 (GND), C7.2, TP5.1, TP7.1, TP9.1
- net VBUS0: now also TP1.1
- net VBUS1: now also TP6.1
- net RGB: now reaches U1.30 (SPIDQS/GPIO37/FSPIQ/SUBSPIQ)
- net RGB: now also U3.3 (DI)

Commit message: ProtoboardSmall : Add QWIIC connector + switch USB C label
Parts:
- added J12: Qwiic_Vertical, SparkFun-Connector:JST04_1MM_Vertical, symbol SparkFun-Connector:Qwiic_Vertical
- added R6, R7: 10K, Resistor_SMD:R_0402_1005Metric, symbol Device:R
Connections:
- net +3V3: now also J12.2 (Pin_2), R6.2, R7.2
- net GND: now also J12.1 (Pin_1)
- net I2C_SCL: now reaches U1.17 (GPIO9/TOUCH9/ADC1_CH8/FSPIHD/SUBSPIHD)
- net I2C_SCL: now also J12.4 (Pin_4), R7.1
- net I2C_SDA: now reaches U1.18 (GPIO10/TOUCH10/ADC1_CH9/FSPICS0/FSPIIO4/SUBSPICS0)
- net I2C_SDA: now also J12.3 (Pin_3), R6.1
- new net: J12.NC1 (NC), J12.NC2 (NC)
- no-connect marks 19 -> 17
Changed lines of the file:
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@@
   (junction (at 21.8948 27.94) (diameter 0) (color 0 0 0 0)
+  )
+  (junction (at 97.79 139.7) (diameter 0) (color 0 0 0 0)
   )
   (junction (at 197.5612 39.497) (diameter 0) (color 0 0 0 0)
@@
   (no_connect (at 215.265 152.4))
   (no_connect (at 156.21 45.72))
-  (no_connect (at 41.91 55.88))
-  (no_connect (at 41.91 53.34))
   (no_connect (at 156.21 60.96))
   (no_connect (at 156.21 58.42))
@@
     (stroke (width 0) (type default))
   )
+  (wire (pts (xy 97.79 139.7) (xy 97.79 140.97))
+    (stroke (width 0) (type default))
+  )
   (polyline (pts (xy 180.1368 106.8578) (xy 180.1368 107.061))
     (stroke (width 0) (type default))
@@
     (stroke (width 0) (type default))
   )
+  (wire (pts (xy 97.79 140.97) (xy 95.25 140.97))
+    (stroke (width 0) (type default))
+  )
+  (wire (pts (xy 95.25 138.43) (xy 97.79 138.43))
+    (stroke (width 0) (type default))
+  )
   (wire (pts (xy 260.35 158.75) (xy 267.97 158.75))
     (stroke (width 0) (type default))
@@
     (stroke (width 0) (type default))
   )
+  (wire (pts (xy 97.79 138.43) (xy 97.79 139.7))
+    (stroke (width 0) (type default))
+  )
   (wire (pts (xy 21.8948 27.94) (xy 29.21 27.94))
     (stroke (width 0) (type default))
@@
     (effects (font (size 1.27 1.27)) (justify left bottom))
   )
+  (label "I2C_SDA" (at 130.81 135.89 180) (fields_autoplaced)
+    (effects (font (size 1.27 1.27)) (justify right bottom))
+  )
   (label "COM1" (at 189.23 79.375 180) (fields_autoplaced)
     (effects (font (size 1.27 1.27)) (justify right bottom))
@@
     (effects (font (size 1.27 1.27)) (justify left bottom))
   )
+  (label "I2C_SCL" (at 87.63 140.97 180) (fields_autoplaced)
+    (effects (font (size 1.27 1.27)) (justify right bottom))
+  )
   (label "CH12" (at 214.63 102.235 0) (fields_autoplaced)
     (effects (font (size 1.27 1.27)) (justify left bottom))
@@
     (effects (font (size 1.27 1.27)) (justify right bottom))
   )
+  (label "I2C_SCL" (at 41.91 53.34 180) (fields_autoplaced)
+    (effects (font (size 1.27 1.27)) (justify right bottom))
+  )
   (label "USB1_DP" (at 104.14 175.26 180) (fields_autoplaced)
     (effects (font (size 1.27 1.27)) (justify right bottom))
@@
     (effects (font (size 1.27 1.27)) (justify right bottom))
   )
+  (label "I2C_SDA" (at 41.91 55.88 180) (fields_autoplaced)
+    (effects (font (size 1.27 1.27)) (justify right bottom))
+  )
   (label "CH11" (at 214.63 99.695 0) (fields_autoplaced)
     (effects (font (size 1.27 1.27)) (justify left bottom))
@@
   (label "VBUS0" (at 66.04 167.005 0) (fields_autoplaced)
     (effects (font (size 1.27 1.27)) (justify left bottom))
+  )
+  (label "I2C_SDA" (at 87.63 138.43 180) (fields_autoplaced)
+    (effects (font (size 1.27 1.27)) (justify right bottom))
+  )
+  (label "I2C_SCL" (at 130.81 133.35 180) (fields_autoplaced)
+    (effects (font (size 1.27 1.27)) (justify right bottom))
   )
   (symbol (lib_id "power:+3.3V") (at 232.41 67.31 90) (unit 1)
@@
         (path "/f2571a4c-3e67-4916-9c0e-b0974b924c84"
           (reference "#PWR0106") (unit 1)
+        )
+      )
+    )
+  )
+  (symbol (lib_id "SparkFun-Connector:Qwiic_Vertical") (at 135.89 135.89 0) (unit 1)
+    (in_bom yes) (on_board yes) (dnp no) (fields_autoplaced)
+    (property "Reference" "J12" (at 144.78 135.89 0)
+      (effects (font (size 1.27 1.27)) (justify left))
+    )
+    (property "Value" "Qwiic_Vertical" (at 144.78 138.43 0)
+      (effects (font (size 1.27 1.27)) (justify left))
+    )
+    (property "Footprint" "SparkFun-Connector:JST04_1MM_Vertical" (at 135.89 148.59 0)
+      (effects (font (size 1.27 1.27)) hide)
+    )
+    (property "Datasheet" "https://www.jst-mfg.com/product/pdf/eng/eSH.pdf" (at 135.89 151.13 0)
+      (effects (font (size 1.27 1.27)) hide)
+    )
+    (property "PROD_ID" "CONN-14483" (at 135.89 146.05 0)
+      (effects (font (size 1.27 1.27)) hide)
+    )
+    (property "LCSC" "C160390" (at 135.89 135.89 0)
+      (effects (font (size 1.27 1.27)) hide)
+    )
+    (pin "1")
+    (pin "2")
+    (pin "3")
+    (pin "4")
+    (pin "NC1")
+    (pin "NC2")
+    (instances
+      (project "ProtoBoardSESmall"
+        (path "/f2571a4c-3e67-4916-9c0e-b0974b924c84"
+          (reference "J12") (unit 1)
         )
       )
@@
     )
   )
+  (symbol (lib_id "power:+3.3V") (at 130.81 138.43 90) (unit 1)
+    (in_bom yes) (on_board yes) (dnp no) (fields_autoplaced)
+    (property "Reference" "#PWR09" (at 134.62 138.43 0)
+      (effects (font (size 1.27 1.27)) hide)
+    )
+    (property "Value" "+3.3V" (at 127.4572 138.4299 90)
+      (effects (font (size 1.27 1.27)) (justify left))
+    )
+    (property "Footprint" "" (at 130.81 138.43 0)
+      (effects (font (size 1.27 1.27)) hide)
+    )
+    (property "Datasheet" "" (at 130.81 138.43 0)
+      (effects (font (size 1.27 1.27)) hide)
+    )
+    (pin "1")
+    (instances
+      (project "ProtoBoardSESmall"
+        (path "/f2571a4c-3e67-4916-9c0e-b0974b924c84"
+          (reference "#PWR09") (unit 1)
+        )
+      )
+    )
+  )
   (symbol (lib_id "power:GND") (at 147.32 180.34 90) (unit 1)
     (in_bom yes) (on_board yes) (dnp no) (fields_autoplaced)
@@
     )
   )
+  (symbol (lib_id "power:GND") (at 130.81 140.97 270) (unit 1)
+    (in_bom yes) (on_board yes) (dnp no) (fields_autoplaced)
+    (property "Reference" "#PWR010" (at 124.46 140.97 0)
+      (effects (font (size 1.27 1.27)) hide)
+    )
+    (property "Value" "GND" (at 127.635 140.9699 90)
+      (effects (font (size 1.27 1.27)) (justify right))
+    )
+    (property "Footprint" "" (at 130.81 140.97 0)
+      (effects (font (size 1.27 1.27)) hide)
+    )
+    (property "Datasheet" "" (at 130.81 140.97 0)
+      (effects (font (size 1.27 1.27)) hide)
+    )
+    (pin "1")
+    (instances
+      (project "ProtoBoardSESmall"
+        (path "/f2571a4c-3e67-4916-9c0e-b0974b924c84"
+          (reference "#PWR010") (unit 1)
+        )
+      )
+    )
+  )
   (symbol (lib_id "BM05B-SRSS-TB_LF__SN_:BM05B-SRSS-TB_LF__SN_") (at 273.685 66.04 0) (unit 1)
     (in_bom yes) (on_board yes) (dnp no)
@@
     )
   )
+  (symbol (lib_id "power:+3.3V") (at 97.79 139.7 270) (unit 1)
+    (in_bom yes) (on_board yes) (dnp no) (fields_autoplaced)
+    (property "Reference" "#PWR011" (at 93.98 139.7 0)
+      (effects (font (size 1.27 1.27)) hide)
+    )
+    (property "Value" "+3.3V" (at 101.6 139.7 90)
+      (effects (font (size 1.27 1.27)) (justify left))
+    )
+    (property "Footprint" "" (at 97.79 139.7 0)
+      (effects (font (size 1.27 1.27)) hide)
+    )
+    (property "Datasheet" "" (at 97.79 139.7 0)
+      (effects (font (size 1.27 1.27)) hide)
+    )
+    (pin "1")
+    (instances
+      (project "ProtoBoardSESmall"
+        (path "/f2571a4c-3e67-4916-9c0e-b0974b924c84"
+          (reference "#PWR011") (unit 1)
+        )
+      )
+    )
+  )
   (symbol (lib_id "Switch:SW_Push") (at 122.555 127.635 0) (unit 1)
     (in_bom yes) (on_board yes) (dnp no) (fields_autoplaced)
@@
     )
   )
+  (symbol (lib_id "Device:R") (at 91.44 138.43 90) (unit 1)
+    (in_bom yes) (on_board yes) (dnp no)
+    (property "Reference" "R6" (at 95.25 137.16 90)
+      (effects (font (size 1.27 1.27)))
+    )
+    (property "Value" "10K" (at 91.44 138.43 90)
+      (effects (font (size 1.27 1.27)))
+    )
+    (property "Footprint" "Resistor_SMD:R_0402_1005Metric" (at 91.44 140.208 90)
+      (effects (font (size 1.27 1.27)) hide)
+    )
+    (property "Datasheet" "~" (at 91.44 138.43 0)
+      (effects (font (size 1.27 1.27)) hide)
+    )
+    (property "LCSC" "C60490" (at 91.44 138.43 90)
+      (effects (font (size 1.27 1.27)) hide)
+    )
+    (pin "1")
+    (pin "2")
+    (instances
+      (project "ProtoBoardSESmall"
+        (path "/f2571a4c-3e67-4916-9c0e-b0974b924c84"
+          (reference "R6") (unit 1)
+        )
+      )
+    )
+  )
   (symbol (lib_id "Connector:TestPoint") (at 154.305 153.67 270) (unit 1)
     (in_bom yes) (on_board yes) (dnp no)
@@
         )
       )
+    )
+  )
+  (symbol (lib_id "Device:R") (at 91.44 140.97 90) (unit 1)
+    (in_bom yes) (on_board yes) (dnp no)
+    (property "Reference" "R7" (at 95.25 139.7 90)
+      (effects (font (size 1.27 1.27)))
+    )
+    (property "Value" "10K" (at 91.44 140.97 90)
+      (effects (font (size 1.27 1.27)))
+    )
+    (property "Footprint" "Resistor_SMD:R_0402_1005Metric" (at 91.44 142.748 90)
+      (effects (font (size 1.27 1.27)) hide)
+    )
+    (property "Datasheet" "~" (at 91.44 140.97 0)
+      (effects (font (size 1.27 1.27)) hide)
+    )
+    (property "LCSC" "C60490" (at 91.44 140.97 90)
+      (effects (font (size 1.27 1.27)) hide)
+    )
+    (pin "1")
+    (pin "2")
+    (instances
+      (project "ProtoBoardSESmall"
+        (path "/f2571a4c-3e67-4916-9c0e-b0974b924c84"
+          (reference "R7") (unit 1)
+        )
+      )
